File: design_files/AST1028.brd (EAGLE design)
At the start: 12 x 12 mm, 4 parts, among them J1 SM05B, J3 FSM8JSMA

Commit message: name update
Parts:
- renumbered J3 to J2
Other:
- board text added: "Wireling Large Button"
- board text removed: "Large Pushbutton Board"
Changed lines of the file:
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@@
 <layer number="54" name="bGND_GNDA" color="7" fill="1" visible="yes" active="yes"/>
 <layer number="56" name="wert" color="7" fill="1" visible="yes" active="yes"/>
+<layer number="57" name="tCAD" color="7" fill="1" visible="no" active="no"/>
+<layer number="58" name="bCAD" color="7" fill="1" visible="no" active="no"/>
+<layer number="59" name="Invisible" color="7" fill="1" visible="no" active="no"/>
+<layer number="61" name="stand" color="7" fill="1" visible="no" active="no"/>
+<layer number="88" name="SimResults" color="9" fill="1" visible="yes" active="yes"/>
+<layer number="89" name="SimProbes" color="9" fill="1" visible="yes" active="yes"/>
+<layer number="90" name="Modules" color="5" fill="1" visible="yes" active="yes"/>
 <layer number="91" name="Nets" color="2" fill="1" visible="no" active="no"/>
 <layer number="92" name="Busses" color="1" fill="1" visible="no" active="no"/>
@@
 <layer number="97" name="Info" color="7" fill="1" visible="no" active="no"/>
 <layer number="98" name="Guide" color="6" fill="1" visible="no" active="no"/>
+<layer number="99" name="SpiceOrder" color="5" fill="1" visible="no" active="no"/>
 <layer number="100" name="Muster" color="7" fill="1" visible="yes" active="yes"/>
 <layer number="101" name="Patch_Top" color="7" fill="1" visible="yes" active="yes"/>
@@
 <layer number="111" name="tGTest" color="4" fill="1" visible="no" active="no"/>
 <layer number="112" name="bGTest" color="1" fill="1" visible="no" active="no"/>
+<layer number="113" name="HENWAY_PKG" color="12" fill="1" visible="yes" active="yes"/>
+<layer number="114" name="50_Electronics_Plate" color="7" fill="1" visible="yes" active="yes"/>
+<layer number="115" name="henwayRES" color="5" fill="1" visible="yes" active="yes"/>
 <layer number="116" name="Patch_BOT" color="7" fill="1" visible="yes" active="yes"/>
 <layer number="117" name="mPads" color="7" fill="1" visible="no" active="no"/>
@@
 <layer number="151" name="HeatSink" color="7" fill="1" visible="yes" active="yes"/>
 <layer number="152" name="mbDocu" color="7" fill="1" visible="no" active="no"/>
+<layer number="153" name="FabDoc1" color="6" fill="1" visible="no" active="no"/>
+<layer number="154" name="FabDoc2" color="2" fill="1" visible="no" active="no"/>
+<layer number="155" name="FabDoc3" color="7" fill="15" visible="no" active="no"/>
+<layer number="156" name="bCapacitor" color="7" fill="1" visible="yes" active="yes"/>
+<layer number="157" name="tResistor" color="7" fill="1" visible="yes" active="yes"/>
+<layer number="158" name="bResistor" color="7" fill="1" visible="yes" active="yes"/>
+<layer number="159" name="henwayCAP" color="13" fill="1" visible="yes" active="yes"/>
+<layer number="160" name="IDFDebug" color="7" fill="1" visible="yes" active="yes"/>
 <layer number="191" name="mNets" color="7" fill="1" visible="no" active="no"/>
 <layer number="192" name="mBusses" color="7" fill="1" visible="no" active="no"/>
@@
 <layer number="223" name="223bmp" color="7" fill="1" visible="yes" active="yes"/>
 <layer number="224" name="224bmp" color="7" fill="1" visible="yes" active="yes"/>
+<layer number="231" name="Eagle3D_PG1" color="7" fill="1" visible="yes" active="yes"/>
+<layer number="232" name="Eagle3D_PG2" color="7" fill="1" visible="yes" active="yes"/>
+<layer number="233" name="Eagle3D_PG3" color="7" fill="1" visible="yes" active="yes"/>
 <layer number="248" name="Housing" color="7" fill="1" visible="yes" active="yes"/>
 <layer number="249" name="Edge" color="7" fill="1" visible="yes" active="yes"/>
@@
 <wire x1="0" y1="40.8" x2="0" y2="0" width="0.127" layer="48"/>
 <dimension x1="14" y1="22" x2="26" y2="22" x3="20" y3="23.454653125" layer="48"/>
-<text x="38.111025" y="4.365003125" size="0.889" layer="48">Large Pushbutton Board</text>
+<text x="38.111025" y="4.365003125" size="0.889" layer="48">Wireling Large Button</text>
 <text x="34.986825" y="1.7714" size="0.889" layer="48">AS-PCB-AST1028</text>
 <text x="57.3810375" y="1.6952" size="0.889" layer="48">1</text>
@@
 <attribute name="VALUE" value="10.0K" x="24.3" y="13.9" size="1.778" layer="27" rot="R270" display="off"/>
 </element>
-<element name="J3" library="tinycircuits" package="SWITCH-FSM/JSM" value="FSM8JSMA" x="20" y="18.6" rot="R90">
+<element name="J2" library="tinycircuits" package="SWITCH-FSM/JSM" value="FSM8JSMA" x="20" y="18.6" rot="R90">
 <attribute name="PARTNO" value="AS-ITM-00278" x="20" y="18.6" size="1.778" layer="27" rot="R90" display="off"/>
 <attribute name="VALUE" value="FSM8JSMA" x="20" y="18.6" size="1.778" layer="27" rot="R90" display="off"/>
@@
 <via x="18.1" y="10.7" extent="1-16" drill="0.381"/>
 <via x="21.9" y="10.7" extent="1-16" drill="0.381"/>
-<contactref element="J3" pad="P$4"/>
-<contactref element="J3" pad="P$1"/>
+<contactref element="J2" pad="P$4"/>
+<contactref element="J2" pad="P$1"/>
 <via x="19" y="19" extent="1-16" drill="0.381"/>
 </signal>
@@
 <wire x1="22" y1="14.6" x2="21.975" y2="14.6" width="0.4064" layer="1"/>
 <wire x1="22" y1="14.5" x2="22" y2="14.6" width="0.4064" layer="1"/>
-<contactref element="J3" pad="P$3"/>
-<contactref element="J3" pad="P$2"/>
+<contactref element="J2" pad="P$3"/>
+<contactref element="J2" pad="P$2"/>
 <wire x1="15.4" y1="20.85" x2="21.975" y2="20.85" width="0.4064" layer="1"/>
 <contactref element="R1" pad="1"/>

Commit message: updated documentation
Parts:
- J1: device tinycircuits:JST_SH_5X1 -> tinycircuits:JST_SH_5X1_EDGE
Changed lines of the file:
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@@
 <attribute name="NO_BOM" value="TRUE" x="34" y="0" size="1.778" layer="27" display="off"/>
 </element>
-<element name="J1" library="tinycircuits" package="JST_SH_5X1" value="SM05B" x="20" y="12.125">
+<element name="J1" library="tinycircuits" package="JST_SH_5X1_EDGE" value="SM05B" x="20" y="12.125">
 <attribute name="PARTNO" value="AS-ITM-00340" x="20" y="12.125" size="1.778" layer="27" display="off"/>
 <attribute name="VALUE" value="SM05B" x="20" y="12.125" size="1.778" layer="27" display="off"/>
