File: design_files/AST1028.sch (EAGLE design)
At the start: 3 parts, among them J1 SM05B, J3 FSM8JSMA

Commit message: name update
Parts:
- renumbered J3 to J2
Other:
- note added: "Hand Populated: -"
- note added: "Hand Soldered: -"
- note added: "Non Populated: -"
- note added: "Notes: -"
- note added: "Variant: Standard - R"
- note added: "Wireling Large Button"
- note removed: "Large Pushbutton Board"
- note removed: "NOTES:"
- moved on the sheet: R1

Commit message: updated documentation
Parts:
- J1: device tinycircuits:AS-ITM-00340 -> tinycircuits:AS-ITM-00340EDGE
Changed lines of the file:
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@@
 <parts>
 <part name="FRAME1" library="tinycircuits" deviceset="FRAME_TINYCIRCUITS_B_L" device=""/>
-<part name="J1" library="tinycircuits" deviceset="AS-ITM-00340" device="" value="SM05B"/>
+<part name="J1" library="tinycircuits" deviceset="AS-ITM-00340" device="EDGE" value="SM05B"/>
 <part name="GND2" library="tinycircuits" deviceset="GND" device=""/>
 <part name="R1" library="tinycircuits" deviceset="AS-ITM-00032" device="" value="10.0K"/>
